File: HW4/HW4-1/HW4-1.kicad_pcb (KiCad board)
At the start: 2 copper layers, 50 x 50 mm, 23 parts, among them J1 Battery, J4 CP2102, SW1 USER, SW2 Slide Switch, SW3 USER, U1 AP7381_33

Commit message: HW5 Done
Parts:
- moved J4 75.3 mm to (64.8, 37.9)
- moved C1 75.1 mm to (61.1, 58.1)
- moved C3 75.1 mm to (61.1, 45.4)
- moved C5 75.1 mm to (61.1, 65.7)
- moved D1 75.1 mm to (33.2, 81.0)
- moved D3 75.1 mm to (40.8, 81.0)
- moved J1 75.1 mm to (31.9, 37.8)
- moved R2 75.1 mm to (61.1, 78.4)
- moved R3 75.1 mm to (35.7, 73.4)
- moved R4 75.1 mm to (33.2, 55.6)
- moved R5 75.1 mm to (37.0, 53.0)
- moved SW1 75.1 mm to (40.8, 60.7)
- moved SW3 75.1 mm to (40.8, 45.4)
- moved U1 75.1 mm to (68.7, 37.8)
- moved U2 75.1 mm to (48.4, 45.4)
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Routing:
- added copper zone on F.Cu, net (none)
